File: hardware/RP-008173-DS-1-CM4IO-KiCAD/CM4IOv5.kicad_sch (KiCad schematic)
At the start: 8 parts

Commit message: added current project
Other:
- removed sheet PCIe-connector
- note removed: "Connector ------ PCIe x1"
