File: hardware/RP-008173-DS-1-CM4IO-KiCAD/CM4_GPIO.kicad_sch (KiCad schematic)
At the start: 28 parts, among them J1 Conn_01x03, J2 Conn_02x07_Odd_Even, J3 Conn_01x03, J7 Micro_SD_Card_Det, J8 THD-20-R, J9 THD-02-R, U1 TPD4EUSB30, U18 RT9742GGJ5, U2 TPD4EUSB30, U3 MagJack-A70-112-331N126, U5 74LVC1G07SE-7, U9 74LVC1G07SE-7

Commit message: added current project
Parts:
- removed J8: THD-20-R, Connector_PinHeader_2.54mm:PinHeader_2x20_P2.54mm_Vertical, symbol Connector_Generic:Conn_02x20_Odd_Even
Other:
- note removed: "40Way GPIO Header"
