File: hardware/RP-008173-DS-1-CM4IO-KiCAD/CM4_HighSpeed.kicad_sch (KiCad schematic)
At the start: 13 parts, among them J10 690-019-298-412, J15 Conn_01x22_Female, J16 Conn_01x22_Female, J22 690-019-298-412, J4 Conn_01x22_Female, J5 Conn_01x22_Female, J6 THD-02-R, U12 RT9742SNGV

Commit message: added current project
Parts:
- removed C12, C13: 100n, Capacitor_SMD:C_0402_1005Metric, symbol Device:C
- removed J10, J22: 690-019-298-412, CM4IO:EDAC 690-019-298-412, symbol CM4IO:HDMI_A_1.4
- removed J15, J16, J4, J5: Conn_01x22_Female, CM4IO:Hirose_FH12-22S-0.5SH_1x22-1MP_P0.50mm_Horizontal, symbol Connector:Conn_01x22_Female
- removed U12: RT9742SNGV, Package_TO_SOT_SMD:SOT-23, symbol CM4IO:RT9742SNGV
Connections:
- no-connect marks 18 -> 2
Other:
- note removed: "Camera Connectors"
- note removed: "Display Connectors"
